Commit message: finished quadroped

File: body.urdf (robot description, URDF)
Before this commit: robot robot, 3 links, 2 joints
Links:
- added link BackLowerLeg, mass 1; collision box size=0.2 0.2 1; visual box size=0.2 0.2 1
- added link DownLeg, mass 1; collision box size=1 0.2 0.2; visual box size=1 0.2 0.2
- added link DownLowerLeg, mass 1; collision box size=0.2 0.2 1; visual box size=0.2 0.2 1
- added link FrontLowerLeg, mass 1; collision box size=0.2 0.2 1; visual box size=0.2 0.2 1
- added link UpLeg, mass 1; collision box size=1 0.2 0.2; visual box size=1 0.2 0.2
- added link UpLowerLeg, mass 1; collision box size=0.2 0.2 1; visual box size=0.2 0.2 1
- link BackLeg: geometry collision box size=0.2 1 0.2; visual box size=0.2 1 0.2
- link FrontLeg: geometry collision box size=0.2 1 0.2; visual box size=0.2 1 0.2
Joints:
- added joint BackLeg_BackLowerLeg: type revolute, parent BackLeg, child BackLowerLeg, origin xyz=0 -1 0 rpy=0 0 0, axis 0 1 0, limit lower=-3.14159 upper=3.14159 effort=0.0 velocity=0.0
- added joint DownLeg_DownLowerLeg: type revolute, parent DownLeg, child DownLowerLeg, origin xyz=1 0 0 rpy=0 0 0, axis 0 1 0, limit lower=-3.14159 upper=3.14159 effort=0.0 velocity=0.0
- added joint FrontLeg_FrontLowerLeg: type revolute, parent FrontLeg, child FrontLowerLeg, origin xyz=0 1 0 rpy=0 0 0, axis 0 1 0, limit lower=-3.14159 upper=3.14159 effort=0.0 velocity=0.0
- added joint Torso_DownLeg: type revolute, parent Torso, child DownLeg, origin xyz=0.5 0 1 rpy=0 0 0, axis 0 1 0, limit lower=-3.14159 upper=3.14159 effort=0.0 velocity=0.0
- added joint Torso_UpLeg: type revolute, parent Torso, child UpLeg, origin xyz=-0.5 0 1 rpy=0 0 0, axis 0 1 0, limit lower=-3.14159 upper=3.14159 effort=0.0 velocity=0.0
- added joint UpLeg_UpLowerLeg: type revolute, parent UpLeg, child UpLowerLeg, origin xyz=-1 0 0 rpy=0 0 0, axis 0 1 0, limit lower=-3.14159 upper=3.14159 effort=0.0 velocity=0.0
- joint Torso_BackLeg: axis 0 1 0 -> 1 0 0; origin xyz=-0.5 0 1 rpy=0 0 0 -> xyz=0 -0.5 1 rpy=0 0 0
- joint Torso_FrontLeg: axis 0 1 0 -> 1 0 0; origin xyz=0.5 0 1 rpy=0 0 0 -> xyz=0 0.5 1 rpy=0 0 0

Commit message: finalp

File: body.urdf (robot description, URDF)
Before this commit: robot robot, 9 links, 8 joints
Links:
- removed link BackLowerLeg
- removed link DownLowerLeg
- removed link FrontLowerLeg
- removed link UpLowerLeg
- link BackLeg: geometry collision box size=0.2 0.2 1; visual box size=0.2 0.2 1
- link DownLeg: geometry collision box size=0.2 0.2 1; visual box size=0.2 0.2 1
- link FrontLeg: geometry collision box size=0.2 0.2 1; visual box size=0.2 0.2 1
- link Torso: geometry collision box size=2 1.8 1; visual box size=2 1.8 1
- link UpLeg: geometry collision box size=0.2 0.2 1; visual box size=0.2 0.2 1
Joints:
- removed joint BackLeg_BackLowerLeg
- removed joint DownLeg_DownLowerLeg
- removed joint FrontLeg_FrontLowerLeg
- removed joint UpLeg_UpLowerLeg
- joint Torso_BackLeg: axis 1 0 0 -> 0 1 0
- joint Torso_DownLeg: origin xyz=0.5 0 1 rpy=0 0 0 -> xyz=0 -1 1 rpy=0 0 0
- joint Torso_FrontLeg: axis 1 0 0 -> 0 1 0; origin xyz=0 0.5 1 rpy=0 0 0 -> xyz=0.5 0.5 1 rpy=0 0 0
- joint Torso_UpLeg: origin xyz=-0.5 0 1 rpy=0 0 0 -> xyz=0 1 1 rpy=0 0 0

Commit message: fixing bot

File: body.urdf (robot description, URDF)
Before this commit: robot robot, 5 links, 4 joints
Links:
- added link Head, mass 1; collision box size=0.2 0.2 0.2; visual box size=0.2 0.2 0.2
- link BackLeg: geometry collision box size=0.1 0.1 0.4; visual box size=0.1 0.1 0.4
- link DownLeg: geometry collision box size=0.1 0.1 0.4; visual box size=0.1 0.1 0.4
- link FrontLeg: geometry collision box size=0.1 0.1 0.4; visual box size=0.1 0.1 0.4
- link Torso: geometry collision box size=1 0.8 0.5; visual box size=1 0.8 0.5
- link UpLeg: geometry collision box size=0.1 0.1 0.4; visual box size=0.1 0.1 0.4
Joints:
- added joint Torso_Head: type revolute, parent Torso, child Head, origin xyz=0.5 0 1 rpy=0 0 0, axis 0 1 0, limit lower=-3.14159 upper=3.14159 effort=0.0 velocity=0.0

Commit message: fixed axis of rotation

File: body.urdf (robot description, URDF)
Before this commit: robot robot, 6 links, 5 joints
Joints:
- joint Torso_BackLeg: axis 0 1 0 -> 1 0 0
- joint Torso_DownLeg: axis 0 1 0 -> 1 0 0; origin xyz=0 -1 1 rpy=0 0 0 -> xyz=0 -0.5 1 rpy=0 0 0
- joint Torso_FrontLeg: axis 0 1 0 -> 1 0 0; origin xyz=0.5 0.5 1 rpy=0 0 0 -> xyz=0.4 0.5 1 rpy=0 0 0
- joint Torso_UpLeg: axis 0 1 0 -> 1 0 0; origin xyz=0 1 1 rpy=0 0 0 -> xyz=0 0.5 1 rpy=0 0 0
