Commit message: randlen fixed

File: body1.urdf (robot description, URDF)
Before this commit: robot robot, 4 links, 3 joints
Links:
- removed link Box3
- link Box0: geometry collision box size=1.329367022503627 0.6571107360280926 1.586541853763059; visual box size=1.329367022503627 0.6571107360280926 1.586541853763059
- link Box1: geometry collision box size=1.3932341731431679 1.4026449673902612 1.6111802821099683; visual box size=1.3932341731431679 1.4026449673902612 1.6111802821099683
- link Box2: geometry collision box size=1.5646296913838675 1.6704443970731657 0.8411484876022999; visual box size=1.5646296913838675 1.6704443970731657 0.8411484876022999
Joints:
- removed joint Box2_Box3
- joint Box0_Box1: origin xyz=0 1.7870272242725478 0 rpy=0 0 0 -> xyz=0 1.029877851709177 0 rpy=0 0 0
- joint Box1_Box2: origin xyz=0 1.8299577702096141 0 rpy=0 0 0 -> xyz=0 1.5365446822317135 0 rpy=0 0 0
