Commit message: renamed snake

File: body4.urdf (robot description, URDF)
Before this commit: robot robot, 10 links, 9 joints
Links:
- removed link Box8
- removed link Box9
- link Box0: geometry collision box size=1.8475703232099143 1.606591718990829 1.186639222512461; visual box size=1.8475703232099143 1.606591718990829 1.186639222512461
- link Box1: geometry collision box size=1.3574067035108348 0.5186449577657657 0.6584517721746496; visual box size=1.3574067035108348 0.5186449577657657 0.6584517721746496
- link Box2: geometry collision box size=1.2618171902763493 1.4785533197691298 0.9383836594187313; visual box size=1.2618171902763493 1.4785533197691298 0.9383836594187313
- link Box3: geometry collision box size=1.8293820924922675 0.8518002520904642 1.898981107801844; visual box size=1.8293820924922675 0.8518002520904642 1.898981107801844
- link Box4: geometry collision box size=1.7415287670511739 1.6886768713169231 1.678519159012944; visual box size=1.7415287670511739 1.6886768713169231 1.678519159012944
- link Box5: geometry collision box size=0.6965758853843123 1.6100590800066592 1.5916212092334312; visual box size=0.6965758853843123 1.6100590800066592 1.5916212092334312
- link Box6: geometry collision box size=1.7828935595869244 0.89639054843488 1.1627842947326785; visual box size=1.7828935595869244 0.89639054843488 1.1627842947326785
- link Box7: geometry collision box size=0.945260471319533 0.6567955081118523 1.3514238276357855; visual box size=0.945260471319533 0.6567955081118523 1.3514238276357855
Joints:
- removed joint Box7_Box8
- removed joint Box8_Box9
- joint Box0_Box1: origin xyz=0 1.7098701249136659 0 rpy=0 0 0 -> xyz=0 1.0626183383782974 0 rpy=0 0 0
- joint Box1_Box2: origin xyz=0 1.5775896404694176 0 rpy=0 0 0 -> xyz=0 0.9985991387674478 0 rpy=0 0 0
- joint Box2_Box3: origin xyz=0 1.3106555070551429 0 rpy=0 0 0 -> xyz=0 1.165176785929797 0 rpy=0 0 0
- joint Box3_Box4: origin xyz=0 1.3917175426628796 0 rpy=0 0 0 -> xyz=0 1.2702385617036938 0 rpy=0 0 0
- joint Box4_Box5: origin xyz=0 1.0450421540731645 0 rpy=0 0 0 -> xyz=0 1.6493679756617912 0 rpy=0 0 0
- joint Box5_Box6: origin xyz=0 0.8281363776380342 0 rpy=0 0 0 -> xyz=0 1.2532248142207696 0 rpy=0 0 0
- joint Box6_Box7: origin xyz=0 1.4001882923318123 0 rpy=0 0 0 -> xyz=0 0.7765930282733662 0 rpy=0 0 0
