Commit message: pretty much done

File: body0.urdf (robot description, URDF)
Before this commit: robot robot, 13 links, 12 joints
Links:
- removed link Box12
- removed link Box13
- removed link Box14
- removed link Box15
- added link Box10, mass 1; collision box size=0.6441418915446661 0.32470198798023436 0.4748146190416233; visual box size=0.6441418915446661 0.32470198798023436 0.4748146190416233
- added link Box11, mass 1; collision box size=0.47517303812662065 0.3478747500004188 0.4826389837133885; visual box size=0.47517303812662065 0.3478747500004188 0.4826389837133885
- added link Box5, mass 1; collision box size=0.35420941406139117 0.42525053139835534 0.496670182042177; visual box size=0.35420941406139117 0.42525053139835534 0.496670182042177
- link Box0: geometry collision box size=0.6354863568074597 0.6840307799240775 0.6717876190180878; visual box size=0.6354863568074597 0.6840307799240775 0.6717876190180878
- link Box1: geometry collision box size=0.2434877030516176 0.37577488031071593 0.2087572219137685; visual box size=0.2434877030516176 0.37577488031071593 0.2087572219137685
- link Box2: geometry collision box size=0.21308516287086693 0.6411954281624346 0.5249562687199247; visual box size=0.21308516287086693 0.6411954281624346 0.5249562687199247
- link Box3: geometry collision box size=0.4470501061721919 0.6459476077478138 0.26962024166876514; visual box size=0.4470501061721919 0.6459476077478138 0.26962024166876514
- link Box4: geometry collision box size=0.5298892769706265 0.6548749411656816 0.5550392589030705; visual box size=0.5298892769706265 0.6548749411656816 0.5550392589030705
- link Box6: geometry collision box size=0.22802499349416983 0.541422747031093 0.4639478803909141; visual box size=0.22802499349416983 0.541422747031093 0.4639478803909141
- link Box7: geometry collision box size=0.6530573259336568 0.2800500612537303 0.315912105882729; visual box size=0.6530573259336568 0.2800500612537303 0.315912105882729
- link Box8: geometry collision box size=0.6428926872446574 0.23056809393037175 0.43129134780935574; visual box size=0.6428926872446574 0.23056809393037175 0.43129134780935574
- link Box9: geometry collision box size=0.682386775132422 0.3605643374094475 0.21553306991530002; visual box size=0.682386775132422 0.3605643374094475 0.21553306991530002
Joints:
- removed joint Box0_Box12
- removed joint Box0_Box6
- removed joint Box1_Box13
- removed joint Box1_Box7
- removed joint Box2_Box14
- removed joint Box2_Box8
- removed joint Box3_Box15
- removed joint Box3_Box9
- added joint Box10_Box11: type revolute, parent Box10, child Box11, origin xyz=0 -0.33628836899032655 -0.4787268013775059 rpy=0 0 0, axis 0 0 1, limit lower=-3.14159 upper=3.14159 effort=0.0 velocity=0.0
- added joint Box4_Box5: type revolute, parent Box4, child Box5, origin xyz=0 -0.5400627362820185 -0.5258547204726237 rpy=0 0 0, axis 0 0 1, limit lower=-3.14159 upper=3.14159 effort=0.0 velocity=0.0
- added joint Box5_Box6: type revolute, parent Box5, child Box6, origin xyz=0 -0.4833366392147242 -0.48030903121654556 rpy=0 0 0, axis 0 0 1, limit lower=-3.14159 upper=3.14159 effort=0.0 velocity=0.0
- added joint Box6_Box7: type revolute, parent Box6, child Box7, origin xyz=-0.44054115971391333 0 0.0 rpy=0 0 0, axis 0 0 1, limit lower=-3.14159 upper=3.14159 effort=0.0 velocity=0.0
- added joint Box7_Box8: type revolute, parent Box7, child Box8, origin xyz=-0.6479750065891572 0 0.0 rpy=0 0 0, axis 0 0 1, limit lower=-3.14159 upper=3.14159 effort=0.0 velocity=0.0
- added joint Box8_Box9: type revolute, parent Box8, child Box9, origin xyz=0.6626397311885397 0 0.0 rpy=0 0 0, axis 0 0 1, limit lower=-3.14159 upper=3.14159 effort=0.0 velocity=0.0
- added joint Box9_Box10: type revolute, parent Box9, child Box10, origin xyz=0 -0.3426331626948409 0.34517384447846167 rpy=0 0 0, axis 0 0 1, limit lower=-3.14159 upper=3.14159 effort=0.0 velocity=0.0
- joint Box0_Box1: origin xyz=0 0.4588281090033321 0 rpy=0 0 0 -> xyz=-0.43948702992953864 0 0.0 rpy=0 0 0
- joint Box1_Box2: origin xyz=0 0.34744627064633926 0 rpy=0 0 0 -> xyz=0 -0.5084851542365753 0.36685674531684664 rpy=0 0 0
- joint Box2_Box3: origin xyz=0 0.37064208476739346 0 rpy=0 0 0 -> xyz=0 -0.6435715179551242 0.39728825519434496 rpy=0 0 0
- joint Box3_Box4: origin xyz=0 0.5585427122587804 0 rpy=0 0 0 -> xyz=0.4884696915714092 0 0.4123297502859178 rpy=0 0 0
